File: Keyboard/Numeric Pad/V1/v364mx-numpad.kicad_sch (KiCad schematic)
At the start: 20 parts, among them J9 KEYPAD2, SW193 KP"0", SW29 KP "@", SW30 KP "+", SW31 KP "-" was KP "*", SW32 KP "=", SW45 KP "7", SW46 KP "8", SW47 KP "9", SW48 KP "*", SW61 KP "4", SW62 KP "5", SW63 KP "6", SW64 KP "/", SW77 KP "1", SW78 KP "2", SW79 KP "3", SW80 "ENTER", SW94 KP ".", SW95 KP ":" was KP "00"

Commit message: Fix Numpad V1R1, add gerbers
Fixed some DRC errors, missing traces on schematic and added gerbers. NOTE: V1R2 is available and recommended over this V1R1 update as it gives you the choice to use regular or low-profile switches.
Connections:
- net R0: now also SW78.2
- net R1: now also SW61.2
- net R2: now also SW63.2
