File: PCB/V364.kicad_sch (KiCad schematic)
At the start: 239 parts, among them CN1 Conn_01x04, CN2 Conn_01x07, CN3 Conn_01x07, CN4 50PinEdge, CN5 Conn_01x08, CN6 Conn_01x08, CN7 Conn_01x08, CN8 Keyboard-Matrix, J1 Jumper_NC_Dual, J10 Jumper_NC_Dual, J11 Jumper_NC_Dual, J12 Jumper_NC_Dual, J2 Jumper_NC_Dual, J3 Jumper_NC_Dual, J4 Jumper_NC_Dual, J5 Jumper_NC_Dual, J6 Jumper_NC_Dual, J7 SolderJumper_2_Bridged, J8 SolderJumper_2_Open, J9 SolderJumper_2_Bridged, M1 RFMODULATOR, P1 24PinEdge, Q1 2SC1815, Q2 2SC1815, Q3 2SC1815, Q4 2SD880, Q5 2N2222, SW1 SW_DPST, SW2 SW_Push, U1 8360, U10 74LS257, U11 4164, U12 4164, U13 4164, U14 4164, U15 4164, U16 4164, U17 4164, U18 4164, U19 251641, U2 8501, U20 74LS139, U21 74LS175, U22 74LS27, U23 23128, U24 23128, U25 23128, U26 23128, U27 6529, U28 23128, U29 23128, U3 6551, U30 8706, U31 T6721, U4 74LS08, U5 6529, U6 74LS04, U7 74LS06N, U8 LM555, U9 74LS257, Y1 OPTION, Y2 1.8432M, Y3 640kHz

Commit message: Fix "voice" audio line to output section
Voice will mix with TED sound and cartridge audio.
Connections:
- net EXT_AUDIO: no longer FB8.2, R8.1, R9.2
- net VOICE: now also FB8.2, R8.1, R9.2
Other:
- note added: "Register Select:"
- note added: "STARTED: 2026-09-01 UPDATED: 2026-10-08"
- note added: "Speech ROM"
- note added: "Speech chip output goes here (same as the cartridge port)"
- note removed: "STARTED: 2026-09-01 UPDATED: 2026-09-13"
Changed lines of the file:
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@@
 	(title_block
 		(title "V364 Remake")
-		(date "2026-09-12")
+		(date "2026-10-08")
 		(rev "Bo Proto")
 		(comment 1 "V364 Prototype Remake by Steve J. Gray")
@@
 		)
 	)
+	(text "Speech ROM"
+		(exclude_from_sim no)
+		(at 278.638 51.308 0)
+		(effects
+			(font
+				(size 1.27 1.27)
+			)
+		)
+	)
 	(text "RS-232"
 		(exclude_from_sim no)
@@
 		)
 	)
-	(text "STARTED: 2026-09-01\nUPDATED: 2026-09-13"
+	(text "STARTED: 2026-09-01\nUPDATED: 2026-10-08"
 		(exclude_from_sim no)
 		(at 48.006 400.812 0)
@@
 		)
 	)
+	(text "Speech chip output\ngoes here (same as\nthe cartridge port)"
+		(exclude_from_sim no)
+		(at 340.106 327.152 0)
+		(effects
+			(font
+				(size 1.27 1.27)
+			)
+		)
+	)
 	(text "AUDIO\nVIDEO"
 		(exclude_from_sim no)
@@
 		)
 	)
+	(text "Register Select:"
+		(exclude_from_sim no)
+		(at 317.754 179.07 0)
+		(effects
+			(font
+				(size 1.27 1.27)
+			)
+		)
+	)
 	(junction
 		(at 48.006 310.388)
@@
 		)
 	)
+	(label "Custom Gate Array"
+		(at 82.042 241.046 0)
+		(effects
+			(font
+				(size 1.27 1.27)
+			)
+			(justify left bottom)
+		)
+	)
 	(label "ATN"
 		(at 566.928 330.2 180)
@@
 		)
 	)
-	(global_label "EXT_AUDIO"
+	(global_label "VOICE"
 		(shape input)
 		(at 350.012 322.58 180)
